File: procyon-power-distribution-board/procyon-power-distribution-board.kicad_sch (KiCad schematic)
At the start: 18 parts, among them Q1 BSS138, Q2 AO3401A, Q3 BSS138, Q4 AO3401A, Q5 BSS138, Q6 AO3401A, Q7 BSS138, Q8 AO3401A

Commit message: Mostly Done with Schematic. Need to wire up connectors (JST-XH???) and add some more filtering caps to the INA260
Parts:
- added Q10: AO3401A, Package_TO_SOT_SMD:SOT-23, symbol Transistor_FET:AO3401A
- added Q9: BSS138, Package_TO_SOT_SMD:SOT-23, symbol Transistor_FET:BSS138
- added R10, R11: 2.7k, symbol Device:R
- added R12: 100, Resistor_SMD:R_0603_1608Metric_Pad0.98x0.95mm_HandSolder, symbol Device:R
- added R13: 10k, Resistor_SMD:R_0603_1608Metric_Pad0.98x0.95mm_HandSolder, symbol Device:R
- added U2: INA260, Package_SO:TSSOP-16_4.4x5mm_P0.65mm, symbol Sensor:INA260
Connections:
- net +5V: now also Q10.2 (S), R13.1
- net +BATT: now also U2.1 (IN+), U2.12 (VBUS), U2.14 (IN-), U2.15 (IN-), U2.16 (IN-), U2.2 (IN+), U2.3 (IN+)
- net GND: now also Q9.2 (S), U2.11 (GND), U2.4 (A1), U2.5 (A0), U2.6 (GND)
- new net: Q10.1 (G), R12.1, R13.2
- new net: Q9.3 (D), R12.2
- new net +3V3: R10.1, R11.1, U2.10 (VS)
- new net DC_0_+: Q10.3 (D)
- new net INA_SCL: R10.2, U2.9 (SCL)
- new net INA_SDA: R11.2, U2.8 (SDA)
- new net MCU_DC_0: Q9.1 (G)
- no-connect marks 1 -> 2
Other:
- note added: "INA260 - Current Sensing IC"
- note added: "Place These If DC"
- note added: "Place These if BLDC"
- moved on the sheet: Q1, Q2, Q3, Q4, Q5, Q6, Q7, Q8, R1, R2, R3, R4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

Commit message: Major changes, mostly finished, needs mounting holes and drc then finished.
Parts:
- added C1: 100nF, Capacitor_SMD:C_0603_1608Metric_Pad1.08x0.95mm_HandSolder, symbol Device:C_Small
- added J1: BLDC_Pwr, Connector_JST:JST_XH_S2B-XH-A-1_1x02_P2.50mm_Horizontal, symbol Connector:Conn_01x02_Pin
- added J10: XTRA2_PWR, Connector_JST:JST_XH_S2B-XH-A-1_1x02_P2.50mm_Horizontal, symbol Connector:Conn_01x02_Pin
- added J11: Ctrl_Header, Connector_JST:JST_XH_S6B-XH-A-1_1x06_P2.50mm_Horizontal, symbol Connector:Conn_01x06_Pin
- added J12: BATT_IN, Connector_Wire:SolderWire-1.5sqmm_1x02_P6mm_D1.7mm_OD3mm, symbol Connector:Conn_01x02_Pin
- added J2: FPV1_Pwr, Connector_JST:JST_XH_S2B-XH-A-1_1x02_P2.50mm_Horizontal, symbol Connector:Conn_01x02_Pin
- added J3: BDC_Pwr, Connector_JST:JST_XH_S2B-XH-A-1_1x02_P2.50mm_Horizontal, symbol Connector:Conn_01x02_Pin
- added J4: FPV2_Pwr, Connector_JST:JST_XH_S2B-XH-A-1_1x02_P2.50mm_Horizontal, symbol Connector:Conn_01x02_Pin
- added J5: FPV3_Pwr, Connector_JST:JST_XH_S2B-XH-A-1_1x02_P2.50mm_Horizontal, symbol Connector:Conn_01x02_Pin
- added J6: INA260_Header, Connector_JST:JST_XH_S6B-XH-A-1_1x06_P2.50mm_Horizontal, symbol Connector:Conn_01x06_Pin
- added J7: FC_PWR, Connector_JST:JST_XH_S2B-XH-A-1_1x02_P2.50mm_Horizontal, symbol Connector:Conn_01x02_Pin
- added J8: Radio_PWR, Connector_JST:JST_XH_S2B-XH-A-1_1x02_P2.50mm_Horizontal, symbol Connector:Conn_01x02_Pin
- added J9: XTRA1_PWR, Connector_JST:JST_XH_S2B-XH-A-1_1x02_P2.50mm_Horizontal, symbol Connector:Conn_01x02_Pin
- R12, R3, R5, R7: value 100 -> 220
- R2: value 100 -> 220; footprint Resistor_SMD:R_0603_1608Metric_Pad0.98x0.95mm_HandSolder -> esistor_SMD:R_0603_1608Metric_Pad0.98x0.95mm_HandSolder
Connections:
- net +3V3: now also C1.1, J6.6 (Pin_6)
- net +5V: now also J7.1 (Pin_1), J8.1 (Pin_1), J9.1 (Pin_1)
- net +BATT: now also J10.1 (Pin_1), J12.1 (Pin_1)
- net GND: now also C1.2, J1.2 (Pin_2), J10.2 (Pin_2), J12.2 (Pin_2), J2.2 (Pin_2), J3.2 (Pin_2), J4.2 (Pin_2), J5.2 (Pin_2), J6.1 (Pin_1), J6.3 (Pin_3), J6.5 (Pin_5), J7.2 (Pin_2), J8.2 (Pin_2), J9.2 (Pin_2)
- net MCU_BLDC_1: now also J11.6 (Pin_6)
- net MCU_DC_0: now also J11.2 (Pin_2)
- net MCU_FPV_1: now also J11.3 (Pin_3)
- net MCU_FPV_2: now also J11.4 (Pin_4)
- net MCU_FPV_3: now also J11.5 (Pin_5)
- net BLDC_1_+: no longer names the net of Q8.3 (D)
- net BLDC_1_+: now also J1.1 (Pin_1)
- net DC_0_+: no longer names the net of Q10.3 (D)
- net DC_0_+: now also J3.1 (Pin_1)
- net FPV_1_+: no longer names the net of Q2.3 (D)
- net FPV_1_+: now also J2.1 (Pin_1)
- net FPV_2_+: no longer names the net of Q4.3 (D)
- net FPV_2_+: now also J4.1 (Pin_1)
- net FPV_3_+: no longer names the net of Q6.3 (D)
- net FPV_3_+: now also J5.1 (Pin_1)
- net INA_SCL: no longer names the net of R10.2, U2.9 (SCL)
- net INA_SCL: now also J6.4 (Pin_4)
- net INA_SDA: no longer names the net of R11.2, U2.8 (SDA)
- net INA_SDA: now also J6.2 (Pin_2)
- no-connect marks 2 -> 3
Other:
- note added: "'Always On' Pwr Headers"
- note added: "Finish Connectors (JST-XH potentially) be careful of 2.5 mm not 2.54 mm"
- moved on the sheet: R10, R11, R9, U1, U2

Commit message: V1 DONE!
Parts:
- R10, R11: footprint (none) -> Resistor_SMD:R_0603_1608Metric_Pad0.98x0.95mm_HandSolder
Changed lines of the file:
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@@
 			)
 		)
-		(property "Footprint" ""
+		(property "Footprint" "Resistor_SMD:R_0603_1608Metric_Pad0.98x0.95mm_HandSolder"
 			(at 178.562 133.35 90)
 			(effects
@@
 			)
 		)
-		(property "Footprint" ""
+		(property "Footprint" "Resistor_SMD:R_0603_1608Metric_Pad0.98x0.95mm_HandSolder"
 			(at 182.372 133.35 90)
 			(effects
